Commit message: wip

File: description/models/panda/panda.urdf (robot description, URDF)
Before this commit: robot panda, 14 links, 13 joints
Links:
- link panda_hand: geometry visual mesh filename=file://$(find panda_control)/description/models/panda/meshe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
- link panda_leftfinger: geometry visual mesh filename=file://$(find panda_control)/description/models/panda/meshe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
- link panda_link0: geometry visual mesh filename=file://$(find panda_control)/description/models/panda/meshe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
- link panda_link1: geometry visual mesh filename=file://$(find panda_control)/description/models/panda/meshe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
- link panda_link2: geometry visual mesh filename=file://$(find panda_control)/description/models/panda/meshe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
- link panda_link3: geometry visual mesh filename=file://$(find panda_control)/description/models/panda/meshe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
- link panda_link4: geometry visual mesh filename=file://$(find panda_control)/description/models/panda/meshe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
- link panda_link5: geometry visual mesh filename=file://$(find panda_control)/description/models/panda/meshe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
- link panda_link6: geometry visual mesh filename=file://$(find panda_control)/description/models/panda/meshe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
- link panda_link7: geometry visual mesh filename=file://$(find panda_control)/description/models/panda/meshe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
- link panda_rightfinger: geometry visual mesh filename=file://$(find panda_control)/description/models/panda/meshe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
